Commit message: Add lasers.

File: src/simulation_launcher/urdf/turtlebot3_waffle_1d_laser/robot.urdf (robot description, URDF)
Before this commit: robot turtlebot3_waffle_pi, 8 links, 7 joints
Links:
- removed link dt35_laser_link
- added link back_laser_link, mass 0.0; visual cylinder length=0.02 radius=0.002; visual cylinder length=0.02 radius=0.002
- added link front_laser_link, mass 0.0; visual cylinder length=0.02 radius=0.002; visual cylinder length=0.02 radius=0.002
- added link l_laser_link, mass 0.0; visual cylinder length=0.02 radius=0.002; visual cylinder length=0.02 radius=0.002
- added link lb_laser_link, mass 0.0; visual cylinder length=0.02 radius=0.002; visual cylinder length=0.02 radius=0.002
- added link lf_laser_link, mass 0.0; visual cylinder length=0.02 radius=0.002; visual cylinder length=0.02 radius=0.002
- added link r_laser_link, mass 0.0; visual cylinder length=0.02 radius=0.002; visual cylinder length=0.02 radius=0.002
- added link rb_laser_link, mass 0.0; visual cylinder length=0.02 radius=0.002; visual cylinder length=0.02 radius=0.002
- added link rf_laser_link, mass 0.0; visual cylinder length=0.02 radius=0.002; visual cylinder length=0.02 radius=0.002
- link base_link: mass 1.3729096 -> 3.0
Joints:
- removed joint dt35_laser_joint
- added joint back_laser_joint: type fixed, parent base_link, child back_laser_link, origin xyz=-0.197 0 0.11 rpy=0 0 3.141592653589793
- added joint front_laser_joint: type fixed, parent base_link, child front_laser_link, origin xyz=0.069 0 0.11 rpy=0 0 0.0
- added joint l_laser_joint: type fixed, parent base_link, child l_laser_link, origin xyz=0.0 0.133 0.11 rpy=0 0 1.5707963267948966
- added joint lb_laser_joint: type fixed, parent base_link, child lb_laser_link, origin xyz=-0.197 0.133 0.11 rpy=0 0 2.356194490192345
- added joint lf_laser_joint: type fixed, parent base_link, child lf_laser_link, origin xyz=0.069 0.133 0.11 rpy=0 0 0.7853981633974483
- added joint r_laser_joint: type fixed, parent base_link, child r_laser_link, origin xyz=0.0 -0.133 0.11 rpy=0 0 -1.5707963267948966
- added joint rb_laser_joint: type fixed, parent base_link, child rb_laser_link, origin xyz=-0.197 -0.133 0.11 rpy=0 0 -2.356194490192345
- added joint rf_laser_joint: type fixed, parent base_link, child rf_laser_link, origin xyz=0.069 -0.133 0.11 rpy=0 0 -0.7853981633974483

File: src/simulation_launcher/urdf/turtlebot3_waffle_1d_laser/xacro/dt35.xacro (robot description, xacro)
@@ -1,34 +1,40 @@
 <?xml version="1.0"?>
 <robot xmlns:xacro="http://www.ros.org/wiki/xacro">
-  <xacro:macro name="dt35_macro" params="name parent xyz">
+  <xacro:macro name="dt35_macro" params="name parent x y yaw">
     <joint name="${name}_joint" type="fixed">
       <parent link="${parent}"/>
       <child  link="${name}_link"/>
-      <origin xyz="${xyz}" rpy="0 0 0"/>
+      <origin xyz="${x} ${y} 0.11" rpy="0 0 ${yaw * pi / 180}"/>
     </joint>
     <link name="${name}_link">
       <visual>
-        <origin xyz="0.015 0 -0.0065" rpy="0 0 0"/>
+        <origin xyz="-0.025 0 0" rpy="0 1.57 0"/>
         <geometry>
-          <cylinder radius="0.055" length="0.0315" />
+          <cylinder radius="0.01" length="0.05" />
         </geometry>
       </visual>
-      <collision>
-        <origin xyz="0.015 0 -0.0065" rpy="0 0 0"/>
+      <visual> <!-- front leg -->
+        <origin xyz="-0.008 0 -0.015" rpy="0 0 0"/>
         <geometry>
-          <cylinder radius="0.055" length="0.0315" />
+          <cylinder radius="0.002" length="0.02" />
         </geometry>
-      </collision>
+      </visual>
+      <!-- back leg -->
+      <visual>
+        <origin xyz="-0.04 0 -0.015" rpy="0 0 0"/>
+        <geometry>
+          <cylinder radius="0.002" length="0.02" />
+        </geometry>
+      </visual>
       <inertial>
-        <mass value="0.114" />
+        <mass value="0.0" />
         <origin xyz="0 0 0" />
-        <inertia ixx="0.001" ixy="0.0" ixz="0.0"
-                iyy="0.001" iyz="0.0"
-                izz="0.001" />
+        <inertia ixx="0.0" ixy="0.0" ixz="0.0"
+                iyy="0.0" iyz="0.0"
+                izz="0.0" />
       </inertial>
     </link>
     <gazebo reference="${name}_link">
       <sensor type="ray" name="${name}">
-        <pose>-0.064 0 0.121 0 0 0</pose>
         <visualize>true</visualize>
         <always_on>true</always_on>
@@ -44,5 +50,5 @@
           </scan>
           <range>
-            <min>0.10</min>
+            <min>0.0</min>
             <max>30.0</max>
             <resolution>0.01</resolution>
@@ -54,5 +60,5 @@
           </noise>
         </ray>
-        <plugin name="gazebo_ros_lidar_controller" filename="libgazebo_ros_ray_sensor.so">
+        <plugin name="${name}_plugin" filename="libgazebo_ros_ray_sensor.so">
           <ros>
             <!-- <namespace>/my_robot</namespace> -->

File: src/simulation_launcher/urdf/turtlebot3_waffle_1d_laser/xacro/robot.xacro (robot description, xacro)
@@ -26,5 +26,5 @@
     <inertial>
       <origin xyz="0 0 0" rpy="0 0 0"/>
-      <mass value="1.3729096"/>
+      <mass value="3.0"/>
       <inertia ixx="8.7002718e-03" ixy="-4.7576583e-05" ixz="1.1160499e-04"
                 iyy="8.6195418e-03" iyz="-3.5422299e-06" izz="1.4612727e-02" />
@@ -66,5 +66,12 @@
   <xacro:caster_macro name="caster_back_left" x="-0.177" y="0.064" z="-0.004"/>
   <xacro:imu_macro name="tb3_imu" parent="base_link" xyz="0.0 0 0.068" />
-  <xacro:dt35_macro name="dt35_laser" parent="base_link" xyz="-0.064 0 0.122" />
+  <xacro:dt35_macro name="front_laser" parent="base_link" x="0.069" y="0" yaw="0" />
+  <xacro:dt35_macro name="lf_laser" parent="base_link" x="0.069" y="0.133" yaw="45" />
+  <xacro:dt35_macro name="l_laser" parent="base_link" x="0.0" y="0.133" yaw="90" />
+  <xacro:dt35_macro name="lb_laser" parent="base_link" x="-0.197" y="0.133" yaw="135" />
+  <xacro:dt35_macro name="rf_laser" parent="base_link" x="0.069" y="-0.133" yaw="-45" />
+  <xacro:dt35_macro name="r_laser" parent="base_link" x="0.0" y="-0.133" yaw="-90" />
+  <xacro:dt35_macro name="rb_laser" parent="base_link" x="-0.197" y="-0.133" yaw="-135" />
+  <xacro:dt35_macro name="back_laser" parent="base_link" x="-0.197" y="0" yaw="180" />
   <gazebo>
     <plugin name="turtlebot3_diff_drive" filename="libgazebo_ros_diff_drive.so">

Commit message: Add robot_publisher.

File: src/simulation_launcher/urdf/turtlebot3_waffle_1d_laser/robot.urdf (robot description, URDF)
Before this commit: robot turtlebot3_waffle_1d, 15 links, 14 joints
Joints:
- joint base_joint: child base_link -> base_footprint; origin xyz=0 0 0.010 rpy=0 0 0 -> xyz=0 0 -0.010 rpy=0 0 0; parent base_footprint -> base_link

File: src/simulation_launcher/urdf/turtlebot3_waffle_1d_laser/xacro/robot.xacro (robot description, xacro)
@@ -6,7 +6,7 @@
   <link name="base_footprint"/>
   <joint name="base_joint" type="fixed">
-    <parent link="base_footprint"/>
-    <child link="base_link" />
-    <origin xyz="0 0 0.010" rpy="0 0 0"/>
+    <parent link="base_link"/>
+    <child link="base_footprint"/>
+    <origin xyz="0 0 -0.010" rpy="0 0 0"/>
   </joint>
   <!-- Links and Joints -->

Commit message: Fix robot.urdf and spawn.

File: src/simulation_launcher/urdf/turtlebot3_waffle_1d_laser/robot.urdf (robot description, URDF)
Before this commit: robot turtlebot3_waffle_1d, 15 links, 14 joints
Joints:
- joint base_joint: child base_footprint -> base_link; origin xyz=0 0 -0.010 rpy=0 0 0 -> xyz=0 0 0.010 rpy=0 0 0; parent base_link -> base_footprint

File: src/simulation_launcher/urdf/turtlebot3_waffle_1d_laser/xacro/imu.xacro (robot description, xacro)
@@ -56,4 +56,5 @@
         <plugin name="${name}_plugin" filename="libgazebo_ros_imu_sensor.so">
           <ros>
+            <namespace>waffle_1d</namespace>
             <remapping>~/out:=imu</remapping>
           </ros>

File: src/simulation_launcher/urdf/turtlebot3_waffle_1d_laser/xacro/robot.xacro (robot description, xacro)
@@ -6,7 +6,7 @@
   <link name="base_footprint"/>
   <joint name="base_joint" type="fixed">
-    <parent link="base_link"/>
-    <child link="base_footprint"/>
-    <origin xyz="0 0 -0.010" rpy="0 0 0"/>
+    <parent link="base_footprint"/>
+    <child link="base_link" />
+    <origin xyz="0 0 0.010" rpy="0 0 0"/>
   </joint>
   <!-- Links and Joints -->
@@ -77,5 +77,5 @@
     <plugin name="turtlebot3_diff_drive" filename="libgazebo_ros_diff_drive.so">
       <ros>
-        <!-- <namespace>/tb3</namespace> -->
+        <namespace>waffle_1d</namespace>
       </ros>
       <update_rate>30</update_rate>
