Commit message: Adjustment laser.xacro.

File: src/simulation_launcher/urdf/turtlebot3_waffle_1d_laser/xacro/dt35.xacro (robot description, xacro)
@@ -1,5 +1,5 @@
 <?xml version="1.0"?>
 <robot xmlns:xacro="http://www.ros.org/wiki/xacro">
-  <xacro:macro name="dt35_macro" params="name parent x y yaw">
+  <xacro:macro name="dt35_macro" params="namespace name parent x y yaw">
     <joint name="${name}_joint" type="fixed">
       <parent link="${parent}"/>
@@ -45,10 +45,10 @@
               <samples>1</samples>
               <resolution>1</resolution>
-              <min_angle>0</min_angle>
-              <max_angle>0</max_angle>
+              <min_angle>-0.01</min_angle>
+              <max_angle>0.01</max_angle>
             </horizontal>
           </scan>
           <range>
-            <min>0.0</min>
+            <min>0.1</min>
             <max>30.0</max>
             <resolution>0.01</resolution>
@@ -62,11 +62,10 @@
         <plugin name="${name}_plugin" filename="libgazebo_ros_ray_sensor.so">
           <ros>
-            <!-- <namespace>/my_robot</namespace> -->
-            <remapping>~/out:=range</remapping>
+            <namespace>${namespace}</namespace>
+            <remapping>~/out:=${name}_range</remapping>
           </ros>
           <output_type>sensor_msgs/Range</output_type>
-          <frameName>${name}_link</frameName>
+          <frame_name>${name}_link</frame_name>
           <radiation_type>infrared</radiation_type>
-          <field_of_view>0.008726646259971648</field_of_view>
         </plugin>
       </sensor>

File: src/simulation_launcher/urdf/turtlebot3_waffle_1d_laser/xacro/robot.xacro (robot description, xacro)
@@ -1,4 +1,4 @@
 <?xml version="1.0" ?>
-<robot name="turtlebot3_waffle_pi" xmlns:xacro="http://ros.org/wiki/xacro">
+<robot name="turtlebot3_waffle_1d" xmlns:xacro="http://ros.org/wiki/xacro">
   <xacro:include filename="caster.xacro"/>
   <xacro:include filename="dt35.xacro"/>
@@ -66,12 +66,12 @@
   <xacro:caster_macro name="caster_back_left" x="-0.177" y="0.064" z="-0.004"/>
   <xacro:imu_macro name="tb3_imu" parent="base_link" xyz="0.0 0 0.068" />
-  <xacro:dt35_macro name="front_laser" parent="base_link" x="0.069" y="0" yaw="0" />
-  <xacro:dt35_macro name="lf_laser" parent="base_link" x="0.069" y="0.133" yaw="45" />
-  <xacro:dt35_macro name="l_laser" parent="base_link" x="0.0" y="0.133" yaw="90" />
-  <xacro:dt35_macro name="lb_laser" parent="base_link" x="-0.197" y="0.133" yaw="135" />
-  <xacro:dt35_macro name="rf_laser" parent="base_link" x="0.069" y="-0.133" yaw="-45" />
-  <xacro:dt35_macro name="r_laser" parent="base_link" x="0.0" y="-0.133" yaw="-90" />
-  <xacro:dt35_macro name="rb_laser" parent="base_link" x="-0.197" y="-0.133" yaw="-135" />
-  <xacro:dt35_macro name="back_laser" parent="base_link" x="-0.197" y="0" yaw="180" />
+  <xacro:dt35_macro namespace="waffle_1d" name="front_laser" parent="base_link" x="0.069" y="0" yaw="0" />
+  <xacro:dt35_macro namespace="waffle_1d" name="lf_laser" parent="base_link" x="0.069" y="0.133" yaw="45" />
+  <xacro:dt35_macro namespace="waffle_1d" name="l_laser" parent="base_link" x="0.0" y="0.133" yaw="90" />
+  <xacro:dt35_macro namespace="waffle_1d" name="lb_laser" parent="base_link" x="-0.197" y="0.133" yaw="135" />
+  <xacro:dt35_macro namespace="waffle_1d" name="rf_laser" parent="base_link" x="0.069" y="-0.133" yaw="-45" />
+  <xacro:dt35_macro namespace="waffle_1d" name="r_laser" parent="base_link" x="0.0" y="-0.133" yaw="-90" />
+  <xacro:dt35_macro namespace="waffle_1d" name="rb_laser" parent="base_link" x="-0.197" y="-0.133" yaw="-135" />
+  <xacro:dt35_macro namespace="waffle_1d" name="back_laser" parent="base_link" x="-0.197" y="0" yaw="180" />
   <gazebo>
     <plugin name="turtlebot3_diff_drive" filename="libgazebo_ros_diff_drive.so">

Commit message: offset success.

File: src/simulation_launcher/urdf/turtlebot3_waffle_1d_laser/xacro/dt35.xacro (robot description, xacro)
@@ -1,5 +1,5 @@
 <?xml version="1.0"?>
 <robot xmlns:xacro="http://www.ros.org/wiki/xacro">
-  <xacro:macro name="dt35_macro" params="namespace name parent x y yaw">
+  <xacro:macro name="dt35_macro" params="name parent x y yaw">
     <joint name="${name}_joint" type="fixed">
       <parent link="${parent}"/>
@@ -62,5 +62,4 @@
         <plugin name="${name}_plugin" filename="libgazebo_ros_ray_sensor.so">
           <ros>
-            <namespace>${namespace}</namespace>
             <remapping>~/out:=${name}_range</remapping>
           </ros>

File: src/simulation_launcher/urdf/turtlebot3_waffle_1d_laser/xacro/robot.xacro (robot description, xacro)
@@ -66,16 +66,15 @@
   <xacro:caster_macro name="caster_back_left" x="-0.177" y="0.064" z="-0.004"/>
   <xacro:imu_macro name="tb3_imu" parent="base_link" xyz="0.0 0 0.068" />
-  <xacro:dt35_macro namespace="waffle_1d" name="front_laser" parent="base_link" x="0.069" y="0" yaw="0" />
-  <xacro:dt35_macro namespace="waffle_1d" name="lf_laser" parent="base_link" x="0.069" y="0.133" yaw="45" />
-  <xacro:dt35_macro namespace="waffle_1d" name="l_laser" parent="base_link" x="0.0" y="0.133" yaw="90" />
-  <xacro:dt35_macro namespace="waffle_1d" name="lb_laser" parent="base_link" x="-0.197" y="0.133" yaw="135" />
-  <xacro:dt35_macro namespace="waffle_1d" name="rf_laser" parent="base_link" x="0.069" y="-0.133" yaw="-45" />
-  <xacro:dt35_macro namespace="waffle_1d" name="r_laser" parent="base_link" x="0.0" y="-0.133" yaw="-90" />
-  <xacro:dt35_macro namespace="waffle_1d" name="rb_laser" parent="base_link" x="-0.197" y="-0.133" yaw="-135" />
-  <xacro:dt35_macro namespace="waffle_1d" name="back_laser" parent="base_link" x="-0.197" y="0" yaw="180" />
+  <xacro:dt35_macro name="front_laser" parent="base_link" x="0.069" y="0" yaw="0" />
+  <xacro:dt35_macro name="lf_laser" parent="base_link" x="0.069" y="0.133" yaw="45" />
+  <xacro:dt35_macro name="l_laser" parent="base_link" x="0.0" y="0.133" yaw="90" />
+  <xacro:dt35_macro name="lb_laser" parent="base_link" x="-0.197" y="0.133" yaw="135" />
+  <xacro:dt35_macro name="rf_laser" parent="base_link" x="0.069" y="-0.133" yaw="-45" />
+  <xacro:dt35_macro name="r_laser" parent="base_link" x="0.0" y="-0.133" yaw="-90" />
+  <xacro:dt35_macro name="rb_laser" parent="base_link" x="-0.197" y="-0.133" yaw="-135" />
+  <xacro:dt35_macro name="back_laser" parent="base_link" x="-0.197" y="0" yaw="180" />
   <gazebo>
     <plugin name="turtlebot3_diff_drive" filename="libgazebo_ros_diff_drive.so">
       <ros>
-        <namespace>waffle_1d</namespace>
       </ros>
       <update_rate>30</update_rate>
@@ -102,6 +101,5 @@
     <plugin name="gazebo_ros_p3d" filename="libgazebo_ros_p3d.so">
       <ros>
-        <namespace>waffle_1d</namespace>
-        <remapping>odom:=true_position</remapping>
+        <remapping>odom:=gazebo_position</remapping>
       </ros>
       <body_name>base_footprint</body_name>
